File: switchled.kicad_pcb (KiCad board)
At the start: 4 copper layers, 32 x 26 mm, 4 parts, among them J1 Conn_01x02_Pin, SW1 SW_SPST

Commit message: Alain
Parts:
- D1: footprint LED_THT:LED_D3.0mm_Horizontal_O3.81mm_Z10.0mm -> LED_THT:LED_D3.0mm_Horizontal_O6.35mm_Z10.0mm
- R1: footprint Resistor_THT:R_Axial_DIN0411_L9.9mm_D3.6mm_P12.70mm_Horizontal -> Resistor_SMD:R_0201_0603Metric
- SW1: footprint Button_Switch_THT:SW_SPST_Omron_B3F-40xx -> Button_Switch_SMD:SW_SPST_CK_RS282G05A3
- moved R1 48.4 mm to (73.5, 51.5)
- moved SW1 40.9 mm to (73.5, 44.0)
- moved D1 39.6 mm to (77.6, 51.2), turned to 90 degrees
- moved J1 37.0 mm to (70.0, 48.7)
Routing:
- net Net-(D1-A): track 18.0 -> 4.80 mm
- net +3.3V: track 12.5 -> 1.54 mm, vias 0 -> 1
- net Net-(D1-K): track 13.3 -> 3.91 mm
- net GND: track 0.00 -> 1.07 mm, vias 0 -> 1
Other:
- board size 32 x 26 mm -> 24 x 13 mm
