File: switchled.kicad_sch (KiCad schematic)
At the start: 1 part

Commit message: Alain
Parts:
- added D1: LED, LED_THT:LED_D3.0mm_Horizontal_O6.35mm_Z10.0mm, symbol Device:LED
- added J1: Conn_01x02_Pin, Connector_PinHeader_2.54mm:PinHeader_1x02_P2.54mm_Vertical, symbol Connector:Conn_01x02_Pin
- added SW1: SW_SPST, Button_Switch_SMD:SW_SPST_CK_RS282G05A3, symbol Switch:SW_SPST
- R1: footprint (none) -> Resistor_SMD:R_0201_0603Metric
Connections:
- net at R1.1: now also D1.1 (K)
- net GND: now reaches R1.2
- net GND: now also J1.2 (Pin_2)
- new net: D1.2 (A), SW1.2 (B)
- new net +3.3V: J1.1 (Pin_1), SW1.1 (A)
Other:
- moved on the sheet: R1
